File: _autosave-simple_split.kicad_sch (KiCad schematic)
At the start: 118 parts, among them J1 AudioJack3, J2 Conn_01x02, M1 MountingHole, M2 MountingHole, M3 MountingHole, M4 MountingHole, M5 MountingHole, M6 MountingHole, M7 MountingHole, M8 MountingHole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

Commit message: added 7 keys
14 in total between two sides
-F1-12
-2 multipurpose
Parts:
- renumbered COM_SELECT2 to ExtraButtonsSelect1, Extra_Function_Key to Extra_Function_Key1
Changed lines of the file:
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@@
 		(on_board yes)
 		(dnp no)
-		(property "Reference" "COM_SELECT2"
+		(property "Reference" "ExtraButtonsSelect1"
 			(at 113.792 43.18 0)
 			(effects
@@
 			(project "simple_split"
 				(path "/5b940dc4-a4d4-48b9-851f-bc67a6e52b4f"
-					(reference "COM_SELECT2")
+					(reference "ExtraButtonsSelect1")
 					(unit 1)
 				)
@@
 		(dnp no)
 		(fields_autoplaced yes)
-		(property "Reference" "Extra_Function_Key"
+		(property "Reference" "Extra_Function_Key1"
 			(at 62.23 177.8 0)
 			(effects
@@
 			(project "simple_split"
 				(path "/5b940dc4-a4d4-48b9-851f-bc67a6e52b4f"
-					(reference "Extra_Function_Key")
-					(unit 1)
-				)
+					(reference "Extra_Function_Key1")
+					(unit 1)
+				)
