File: simple_split_MX.kicad_pcb (KiCad board)
At the start: 2 copper layers, 182.1 x 114.5 mm, 120 parts, among them J1 AudioJack3, J2 Conn_01x02, M1 MountingHole, M10 MountingHole, M11 MountingHole, M2 MountingHole, M3 MountingHole, M4 MountingHole, M5 MountingHole, M6 MountingHole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

Commit message: added custom silkscreen
Parts:
- added G***: LOGO, Misc Keyboard Parts:Keyboard Icon, F.Cu at (252.1, 187.5)
- added G***: LOGO, Misc Keyboard Parts:Keyboard Icon, B.Cu at (280.9, 188.5)
Other:
- board text added: "ROYAL SPLIT KEYBOARD {dblquote}THE BOSS{dblquote} Nathan Ford 2024 IEEE BYU"

Commit message: added a new Image
Parts:
- removed the G*** at (252.1, 187.5)
- removed the G*** at (280.9, 188.5)
- added G***: LOGO, Misc Keyboard Parts:GPU Silkscreen, F.Cu at (115.0, 167.0)
- added G***: LOGO, Misc Keyboard Parts:Keyboard Icon Smaller, F.Cu at (255.5, 190.5)
- added G***: LOGO, Misc Keyboard Parts:GPU Silkscreen, B.Cu at (115.0, 167.0)
- added G***: LOGO, Misc Keyboard Parts:Keyboard Icon Smaller, B.Cu at (252.5, 184.0)

Commit message: fixed major problem
Connections:
- Bat+1 pad 3: unconnected-(Bat+1-R-Pad3) -> /Bat-
- GND1 pad 2: /GND -> /Bat-
- GND2 pad 2: unconnected-(GND2-L-Pad2) -> /Bat-
- J1 pad S: /GND -> /Bat-
- R1 pad C: /GND -> /Bat-
- TXD1 pad 2: /Bat- -> /Bat+
- TXD2 pad 3: /Bat- -> /Bat+
- U2 pad 1: /GND -> /Bat-
- VCC1 pad 3: /GND -> /Bat-
Routing:
- net /Bat-: track 105.2 -> 262.2 mm, vias 1 -> 2
- net /GND: track 136.2 -> 0.00 mm, vias 1 -> 0
- net /Bat+: track 118.7 -> 138.4 mm, vias 4 -> 6

Commit message: updated pcb
Parts:
- added R4: 10K, Resistor_THT:R_Axial_DIN0204_L3.6mm_D1.6mm_P7.62mm_Horizontal, F.Cu at (266.7, 190.1)
- added R5: 10K, Resistor_THT:R_Axial_DIN0204_L3.6mm_D1.6mm_P7.62mm_Horizontal, F.Cu at (268.6, 192.8)
Routing:
- net /VCC: track 143.1 -> 153.4 mm
- net /SDA: track 87.3 -> 95.4 mm
- net /SCL: track 78.7 -> 84.4 mm

Commit message: updates
Parts:
- moved M6 5.76 mm to (206.5, 137.5)
- moved M4 0.39 mm to (158.5, 121.5)
Connections:
- U1 pad 10: Net-(SCL1-COM) -> /C
- U1 pad 5: /F -> Net-(SDA1-COM)
- U1 pad 6: /E -> Net-(SCL1-COM)
- U1 pad 7: /D -> /F
- U1 pad 8: /C -> /E
- U1 pad 9: Net-(SDA1-COM) -> /D
Routing:
- net Net-(SCL1-COM): track 9.57 -> 17.3 mm, vias 1 -> 2
- net /C: track 341.7 -> 335.7 mm, vias 8 -> 7
- net /D: track 301.8 -> 296.7 mm
- net /Bat-: track 262.2 -> 266.5 mm
- net /E: track 231.3 -> 227.3 mm
- net /2: track 179.8 -> 182.3 mm
