File: simple_split_MX.kicad_sch (KiCad schematic)
At the start: 120 parts, among them J1 AudioJack3, J2 Conn_01x02, M1 MountingHole, M10 MountingHole, M11 MountingHole, M2 MountingHole, M3 MountingHole, M4 MountingHole, M5 MountingHole, M6 MountingHole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

Commit message: fixed major problem
Connections:
- net GND is gone; now on net Bat-: GND1.2 (L), J1.S, R1.C, U2.1 (GND), VCC1.3 (R)
- net Bat+: now also TXD1.2 (L), TXD2.3 (R)
- net Bat-: now also Bat+1.3 (R), GND2.2 (L); no longer TXD1.2 (L), TXD2.3 (R)
Changed lines of the file:
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@@
+	(wire
+		(pts
+			(xy 306.07 120.65) (xy 302.26 120.65)
+		)
+		(stroke
+			(width 0)
+			(type default)
+		)
+	)
 	(wire
 		(pts
@@
 		)
 	)
+	(label "Bat-"
+		(at 302.26 120.65 180)
+		(fields_autoplaced yes)
+		(effects
+			(font
+				(size 1.27 1.27)
+			)
+			(justify right bottom)
+		)
+	)
 	(label "SCL"
 		(at 287.02 158.75 90)
@@
 	)
 	(label "Bat-"
-		(at 351.79 57.15 0)
+		(at 351.79 46.99 0)
 		(fields_autoplaced yes)
 		(effects
@@
 		)
 	)
+	(label "Bat+"
+		(at 351.79 57.15 0)
+		(fields_autoplaced yes)
+		(effects
+			(font
+				(size 1.27 1.27)
+			)
+			(justify left bottom)
+		)
+	)
 	(label "2"
 		(at 353.06 85.09 0)
@@
 		)
 	)
+	(label "GND"
+		(at 306.07 120.65 0)
+		(fields_autoplaced yes)
+		(effects
+			(font
+				(size 1.27 1.27)
+			)
+			(justify left bottom)
+		)
+	)
 	(label "Rotary_B"
 		(at 336.55 78.74 0)
@@
 	)
 	(label "Bat-"
-		(at 293.37 59.69 180)
+		(at 293.37 49.53 180)
 		(fields_autoplaced yes)
 		(effects
@@
 			)
 			(justify left bottom)
+		)
+	)
+	(label "Bat+"
+		(at 293.37 59.69 180)
+		(fields_autoplaced yes)
+		(effects
+			(font
+				(size 1.27 1.27)
+			)
+			(justify right bottom)
 		)
 	)
@@
 	)
 	(symbol
-		(lib_name "Misc Keyboard Parts:SW_Kali_optional_reversable")
 		(lib_id "Misc Keyboard Parts:SW_Kali_optional_reversable")
 		(at 173.99 143.51 0)

Commit message: updated pcb
Parts:
- added R4, R5: 10K, Resistor_THT:R_Axial_DIN0204_L3.6mm_D1.6mm_P7.62mm_Horizontal, symbol Device:R
Connections:
- net SCL: now also R4.2
- net SDA: now also R5.2
- net VCC: now also R4.1, R5.1
Changed lines of the file:
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@@
+		)
+	)
+	(label "SDA"
+		(at 284.48 139.7 270)
+		(fields_autoplaced yes)
+		(effects
+			(font
+				(size 1.27 1.27)
+			)
+			(justify right bottom)
 		)
 	)
@@
 		)
 	)
+	(label "VCC"
+		(at 274.32 132.08 0)
+		(fields_autoplaced yes)
+		(effects
+			(font
+				(size 1.27 1.27)
+			)
+			(justify left bottom)
+		)
+	)
 	(label "SCL"
 		(at 353.06 90.17 0)
@@
 		)
 	)
+	(label "VCC"
+		(at 284.48 132.08 0)
+		(fields_autoplaced yes)
+		(effects
+			(font
+				(size 1.27 1.27)
+			)
+			(justify left bottom)
+		)
+	)
 	(label "4"
 		(at 240.03 179.07 0)
@@
 	(label "SDA"
 		(at 288.29 82.55 180)
+		(fields_autoplaced yes)
+		(effects
+			(font
+				(size 1.27 1.27)
+			)
+			(justify right bottom)
+		)
+	)
+	(label "SCL"
+		(at 274.32 139.7 270)
 		(fields_autoplaced yes)
 		(effects
@@
 	)
 	(symbol
+		(lib_id "Device:R")
+		(at 274.32 135.89 0)
+		(unit 1)
+		(exclude_from_sim no)
+		(in_bom yes)
+		(on_board yes)
+		(dnp no)
+		(fields_autoplaced yes)
+		(property "Reference" "R4"
+			(at 276.86 134.6199 0)
+			(effects
+				(font
+					(size 1.27 1.27)
+				)
+				(justify left)
+			)
+		)
+		(property "Value" "10K"
+			(at 276.86 137.1599 0)
+			(effects
+				(font
+					(size 1.27 1.27)
+				)
+				(justify left)
+			)
+		)
+		(property "Footprint" "Resistor_THT:R_Axial_DIN0204_L3.6mm_D1.6mm_P7.62mm_Horizontal"
+			(at 272.542 135.89 90)
+			(effects
+				(font
+					(size 1.27 1.27)
+				)
+				(hide yes)
+			)
+		)
+		(property "Datasheet" "~"
+			(at 274.32 135.89 0)
+			(effects
+				(font
+					(size 1.27 1.27)
+				)
+				(hide yes)
+			)
+		)
+		(property "Description" "Resistor"
+			(at 274.32 135.89 0)
+			(effects
+				(font
+					(size 1.27 1.27)
+				)
+				(hide yes)
+			)
+		)
+		(pin "1"
+		)
+		(pin "2"
+		)
+		(instances
+			(project "simple_split_MX"
+				(path "/5b940dc4-a4d4-48b9-851f-bc67a6e52b4f"
+					(reference "R4")
+					(unit 1)
+				)
+			)
+		)
+	)
+	(symbol
 		(lib_id "Device:D")
 		(at 66.04 149.86 90)
@@
 					(unit 1)
 				)
+			)
+		)
+	)
+	(symbol
+		(lib_id "Device:R")
+		(at 284.48 135.89 0)
+		(unit 1)
+		(exclude_from_sim no)
+		(in_bom yes)
+		(on_board yes)
+		(dnp no)
+		(fields_autoplaced yes)
+		(property "Reference" "R5"
+			(at 287.02 134.6199 0)
+			(effects
+				(font
+					(size 1.27 1.27)
+				)
+				(justify left)
+			)
+		)
+		(property "Value" "10K"
+			(at 287.02 137.1599 0)
+			(effects
+				(font
+					(size 1.27 1.27)
+				)
+				(justify left)
+			)
+		)
+		(property "Footprint" "Resistor_THT:R_Axial_DIN0204_L3.6mm_D1.6mm_P7.62mm_Horizontal"
+			(at 282.702 135.89 90)
+			(effects
+				(font
+					(size 1.27 1.27)
+				)
+				(hide yes)
+			)
+		)
+		(property "Datasheet" "~"
+			(at 284.48 135.89 0)
+			(effects
+				(font
+					(size 1.27 1.27)
+				)
+				(hide yes)
+			)
+		)
+		(property "Description" "Resistor"
+			(at 284.48 135.89 0)
+			(effects
+				(font
+					(size 1.27 1.27)
+				)
+				(hide yes)
+			)
+		)
+		(pin "1"
+		)
+		(pin "2"
+		)
+		(instances
+			(project "simple_split_MX"
+				(path "/5b940dc4-a4d4-48b9-851f-bc67a6e52b4f"
+					(reference "R5")
+					(unit 1)
+				)

Commit message: updates
Connections:
- net C: now also U1.10 (7); no longer U1.8 (5)
- net D: now also U1.9 (6); no longer U1.7 (4)
- net E: now also U1.8 (5); no longer U1.6 (3)
- net F: now also U1.7 (4); no longer U1.5 (2)
- net at SCL1.1 (COM): now also U1.6 (3); no longer U1.10 (7)
- net at SDA1.1 (COM): now also U1.5 (2); no longer U1.9 (6)
Other:
- moved on the sheet: SCL1, SDA1
Changed lines of the file:
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@@
 	(wire
 		(pts
+			(xy 298.45 87.63) (xy 302.26 87.63)
+		)
+		(stroke
+			(width 0)
+			(type default)
+		)
+	)
+	(wire
+		(pts
 			(xy 179.07 179.07) (xy 196.85 179.07)
 		)
@@
 	(wire
 		(pts
-			(xy 307.34 76.2) (xy 309.88 76.2)
-		)
-		(stroke
-			(width 0)
-			(type default)
-		)
-	)
-	(wire
-		(pts
 			(xy 307.34 73.66) (xy 309.88 73.66)
 		)
@@
 	(wire
 		(pts
-			(xy 307.34 81.28) (xy 309.88 81.28)
-		)
-		(stroke
-			(width 0)
-			(type default)
-		)
-	)
-	(wire
-		(pts
 			(xy 307.34 68.58) (xy 309.88 68.58)
 		)
@@
 	(wire
 		(pts
+			(xy 302.26 87.63) (xy 302.26 78.74)
+		)
+		(stroke
+			(width 0)
+			(type default)
+		)
+	)
+	(wire
+		(pts
 			(xy 196.85 93.98) (xy 214.63 93.98)
 		)
@@
 	(wire
 		(pts
+			(xy 306.07 77.47) (xy 306.07 76.2)
+		)
+		(stroke
+			(width 0)
+			(type default)
+		)
+	)
+	(wire
+		(pts
 			(xy 132.08 171.45) (xy 132.08 200.66)
 		)
@@
 	(wire
 		(pts
+			(xy 307.34 88.9) (xy 309.88 88.9)
+		)
+		(stroke
+			(width 0)
+			(type default)
+		)
+	)
+	(wire
+		(pts
 			(xy 229.87 185.42) (xy 229.87 184.15)
 		)
@@
 	(wire
 		(pts
-			(xy 161.29 208.28) (xy 179.07 208.28)
+			(xy 302.26 78.74) (xy 309.88 78.74)
 		)
 		(stroke
@@
 	(wire
 		(pts
-			(xy 78.74 121.92) (xy 78.74 137.16)
+			(xy 161.29 208.28) (xy 179.07 208.28)
 		)
 		(stroke
@@
 	(wire
 		(pts
-			(xy 302.26 88.9) (xy 309.88 88.9)
+			(xy 78.74 121.92) (xy 78.74 137.16)
 		)
 		(stroke
@@
 	(wire
 		(pts
+			(xy 306.07 76.2) (xy 309.88 76.2)
+		)
+		(stroke
+			(width 0)
+			(type default)
+		)
+	)
+	(wire
+		(pts
 			(xy 78.74 191.77) (xy 67.31 191.77)
 		)
@@
 	(wire
 		(pts
+			(xy 307.34 86.36) (xy 309.88 86.36)
+		)
+		(stroke
+			(width 0)
+			(type default)
+		)
+	)
+	(wire
+		(pts
 			(xy 196.85 151.13) (xy 214.63 151.13)
 		)
@@
 	(wire
 		(pts
-			(xy 204.47 86.36) (xy 204.47 115.57)
+			(xy 307.34 81.28) (xy 309.88 81.28)
 		)
 		(stroke
@@
 	(wire
 		(pts
-			(xy 302.26 91.44) (xy 302.26 88.9)
+			(xy 204.47 86.36) (xy 204.47 115.57)
 		)
 		(stroke
@@
 	(wire
 		(pts
+			(xy 307.34 83.82) (xy 309.88 83.82)
+		)
+		(stroke
+			(width 0)
+			(type default)
+		)
+	)
+	(wire
+		(pts
 			(xy 307.34 66.04) (xy 307.34 68.58)
 		)
@@
 	(wire
 		(pts
-			(xy 302.26 83.82) (xy 302.26 86.36)
-		)
-		(stroke
-			(width 0)
-			(type default)
-		)
-	)
-	(wire
-		(pts
 			(xy 222.25 86.36) (xy 222.25 115.57)
 		)
@@
 	(wire
 		(pts
+			(xy 300.99 80.01) (xy 300.99 77.47)
+		)
+		(stroke
+			(width 0)
+			(type default)
+		)
+	)
+	(wire
+		(pts
 			(xy 229.87 193.04) (xy 238.76 193.04)
 		)
@@
 	(wire
 		(pts
-			(xy 307.34 78.74) (xy 309.88 78.74)
-		)
-		(stroke
-			(width 0)
-			(type default)
-		)
-	)
-	(wire
-		(pts
-			(xy 307.34 83.82) (xy 309.88 83.82)
+			(xy 229.87 208.28) (xy 231.14 208.28)
 		)
 		(stroke
@@
 	(wire
 		(pts
-			(xy 229.87 208.28) (xy 231.14 208.28)
+			(xy 186.69 193.04) (xy 186.69 171.45)
 		)
 		(stroke
@@
 	(wire
 		(pts
-			(xy 186.69 193.04) (xy 186.69 171.45)
+			(xy 332.74 81.28) (xy 336.55 81.28)
 		)
 		(stroke
@@
 	(wire
 		(pts
-			(xy 332.74 81.28) (xy 336.55 81.28)
+			(xy 232.41 93.98) (xy 240.03 93.98)
 		)
 		(stroke
@@
 	(wire
 		(pts
-			(xy 232.41 93.98) (xy 240.03 93.98)
+			(xy 124.46 93.98) (xy 142.24 93.98)
 		)
 		(stroke
@@
 	(wire
 		(pts
-			(xy 124.46 93.98) (xy 142.24 93.98)
+			(xy 300.99 77.47) (xy 306.07 77.47)
 		)
 		(stroke
@@
 	(wire
 		(pts
-			(xy 302.26 86.36) (xy 309.88 86.36)
+			(xy 298.45 80.01) (xy 300.99 80.01)
 		)
 		(stroke
@@
 	)
 	(label "3"
-		(at 288.29 92.71 180)
+		(at 284.48 88.9 180)
 		(fields_autoplaced yes)
 		(effects
@@
 	)
 	(label "C"
-		(at 307.34 83.82 270)
+		(at 307.34 88.9 270)
 		(fields_autoplaced yes)
 		(effects
@@
 	)
 	(label "SCL"
-		(at 288.29 90.17 180)
+		(at 284.48 86.36 180)
 		(fields_autoplaced yes)
 		(effects
@@
 	)
 	(label "F"
-		(at 307.34 76.2 270)
+		(at 307.34 81.28 270)
 		(fields_autoplaced yes)
 		(effects
@@
 	)
 	(label "E"
-		(at 307.34 78.74 270)
+		(at 307.34 83.82 270)
 		(fields_autoplaced yes)
 		(effects
@@
 	)
 	(label "2"
-		(at 288.29 85.09 180)
+		(at 284.48 81.28 180)
 		(fields_autoplaced yes)
 		(effects
@@
 	)
 	(label "SDA"
-		(at 288.29 82.55 180)
+		(at 284.48 78.74 180)
 		(fields_autoplaced yes)
 		(effects
@@
 	)
 	(label "D"
-		(at 307.34 81.28 270)
+		(at 307.34 86.36 270)
 		(fields_autoplaced yes)
 		(effects
@@
 	(symbol
 		(lib_id "Misc Keyboard Parts:Side_Indicator")
-		(at 294.64 91.44 0)
+		(at 290.83 87.63 0)
 		(unit 1)
 		(exclude_from_sim no)
@@
 		(dnp no)
 		(property "Reference" "SCL1"
-			(at 295.148 87.63 0)
+			(at 291.338 83.82 0)
 			(effects
 				(font
@@
 		)
 		(property "Value" "~"
-			(at 295.275 87.63 0)
+			(at 291.465 83.82 0)
 			(effects
 				(font
@@
 		)
 		(property "Footprint" "Misc Keyboard Parts:Side Indicator - Improved"
-			(at 294.64 91.44 0)
+			(at 290.83 87.63 0)
 			(effects
 				(font
@@
 		)
 		(property "Datasheet" ""
-			(at 294.64 91.44 0)
+			(at 290.83 87.63 0)
 			(effects
 				(font
@@
 		)
 		(property "Description" ""
-			(at 294.64 91.44 0)
+			(at 290.83 87.63 0)
 			(effects
 				(font
@@
 	(symbol
 		(lib_id "Misc Keyboard Parts:Side_Indicator")
-		(at 294.64 83.82 0)
+		(at 290.83 80.01 0)
 		(unit 1)
 		(exclude_from_sim no)
@@
 		(dnp no)
 		(property "Reference" "SDA1"
-			(at 295.148 80.01 0)
+			(at 291.338 76.2 0)
 			(effects
 				(font
@@
 		)
 		(property "Value" "~"
-			(at 295.275 80.01 0)
+			(at 291.465 76.2 0)
 			(effects
 				(font
@@
 		)
 		(property "Footprint" "Misc Keyboard Parts:Side Indicator - Improved"
-			(at 294.64 83.82 0)
+			(at 290.83 80.01 0)
 			(effects
 				(font
@@
 		)
 		(property "Datasheet" ""
-			(at 294.64 83.82 0)
+			(at 290.83 80.01 0)
 			(effects
 				(font
@@
 		)
 		(property "Description" ""
-			(at 294.64 83.82 0)
+			(at 290.83 80.01 0)
 			(effects
 				(font
