File: simple_split.kicad_sch (KiCad schematic)
At the start: 118 parts, among them J1 AudioJack3, J2 Conn_01x02, M1 MountingHole, M2 MountingHole, M3 MountingHole, M4 MountingHole, M5 MountingHole, M6 MountingHole, M7 MountingHole, M8 MountingHole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

Commit message: Finished V6
Parts:
- added M10, M11: MountingHole, MountingHole:MountingHole_2.2mm_M2, symbol Mechanical:MountingHole
- renumbered COM_SELECT2 to ExtraButtonsSelect1, Extra_Function_Key to Extra_Function_Key1
Changed lines of the file:
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@@
 		(on_board yes)
 		(dnp no)
-		(property "Reference" "COM_SELECT2"
+		(property "Reference" "ExtraButtonsSelect1"
 			(at 113.792 43.18 0)
 			(effects
@@
 			(project "simple_split"
 				(path "/5b940dc4-a4d4-48b9-851f-bc67a6e52b4f"
-					(reference "COM_SELECT2")
+					(reference "ExtraButtonsSelect1")
 					(unit 1)
 				)
@@
 		(dnp no)
 		(fields_autoplaced yes)
-		(property "Reference" "Extra_Function_Key"
+		(property "Reference" "Extra_Function_Key1"
 			(at 62.23 177.8 0)
 			(effects
@@
 			(project "simple_split"
 				(path "/5b940dc4-a4d4-48b9-851f-bc67a6e52b4f"
-					(reference "Extra_Function_Key")
+					(reference "Extra_Function_Key1")
 					(unit 1)
 				)
@@
 	)
 	(symbol
+		(lib_id "Mechanical:MountingHole")
+		(at 370.84 215.9 0)
+		(unit 1)
+		(exclude_from_sim yes)
+		(in_bom no)
+		(on_board yes)
+		(dnp no)
+		(fields_autoplaced yes)
+		(property "Reference" "M10"
+			(at 373.38 214.6299 0)
+			(effects
+				(font
+					(size 1.27 1.27)
+				)
+				(justify left)
+			)
+		)
+		(property "Value" "MountingHole"
+			(at 373.38 217.1699 0)
+			(effects
+				(font
+					(size 1.27 1.27)
+				)
+				(justify left)
+			)
+		)
+		(property "Footprint" "MountingHole:MountingHole_2.2mm_M2"
+			(at 370.84 215.9 0)
+			(effects
+				(font
+					(size 1.27 1.27)
+				)
+				(hide yes)
+			)
+		)
+		(property "Datasheet" "~"
+			(at 370.84 215.9 0)
+			(effects
+				(font
+					(size 1.27 1.27)
+				)
+				(hide yes)
+			)
+		)
+		(property "Description" "Mounting Hole without connection"
+			(at 370.84 215.9 0)
+			(effects
+				(font
+					(size 1.27 1.27)
+				)
+				(hide yes)
+			)
+		)
+		(instances
+			(project "simple_split"
+				(path "/5b940dc4-a4d4-48b9-851f-bc67a6e52b4f"
+					(reference "M10")
+					(unit 1)
+				)
+			)
+		)
+	)
+	(symbol
 		(lib_id "Mechanical:DIN_Rail_Adapter")
 		(at 309.88 247.65 0)
@@
 					(unit 1)
 				)
+			)
+		)
+	)
+	(symbol
+		(lib_id "Mechanical:MountingHole")
+		(at 388.62 210.82 0)
+		(unit 1)
+		(exclude_from_sim yes)
+		(in_bom no)
+		(on_board yes)
+		(dnp no)
+		(fields_autoplaced yes)
+		(property "Reference" "M11"
+			(at 391.16 209.5499 0)
+			(effects
+				(font
+					(size 1.27 1.27)
+				)
+				(justify left)
+			)
+		)
+		(property "Value" "MountingHole"
+			(at 391.16 212.0899 0)
+			(effects
+				(font
+					(size 1.27 1.27)
+				)
+				(justify left)
+			)
+		)
+		(property "Footprint" "MountingHole:MountingHole_2.2mm_M2"
+			(at 388.62 210.82 0)
+			(effects
+				(font
+					(size 1.27 1.27)
+				)
+				(hide yes)
+			)
+		)
+		(property "Datasheet" "~"
+			(at 388.62 210.82 0)
+			(effects
+				(font
+					(size 1.27 1.27)
+				)
+				(hide yes)
+			)
+		)
+		(property "Description" "Mounting Hole without connection"
+			(at 388.62 210.82 0)
+			(effects
+				(font
+					(size 1.27 1.27)
+				)
+				(hide yes)
+			)
+		)
+		(instances
+			(project "simple_split"
+				(path "/5b940dc4-a4d4-48b9-851f-bc67a6e52b4f"
+					(reference "M11")
+					(unit 1)
+				)

Commit message: added labels
Other:
- company: (none) -> Nathan Ford
- title: (none) -> Split Mechanical Keybard
Changed lines of the file:
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@@
 	(generator_version "8.0")
 	(paper "A3")
+	(title_block
+		(title "Split Mechanical Keybard")
+		(rev "13")
+		(company "Nathan Ford")
+	)
 	(junction
 		(at 78.74 73.66)
@@
 	)
 	(symbol
-		(lib_name "Misc Keyboard Parts:SW_Kali_optional_reversable")
 		(lib_id "Misc Keyboard Parts:SW_Kali_optional_reversable")
 		(at 137.16 143.51 0)
@@
 	)
 	(symbol
-		(lib_name "Misc Keyboard Parts:SW_Kali_optional_reversable")
 		(lib_id "Misc Keyboard Parts:SW_Kali_optional_reversable")
 		(at 191.77 86.36 0)
@@
 	)
 	(symbol
-		(lib_name "Misc Keyboard Parts:SW_Kali_optional_reversable")
 		(lib_id "Misc Keyboard Parts:SW_Kali_optional_reversable")
 		(at 209.55 86.36 0)
@@
 	)
 	(symbol
-		(lib_name "Misc Keyboard Parts:SW_Kali_optional_reversable")
 		(lib_id "Misc Keyboard Parts:SW_Kali_optional_reversable")
 		(at 173.99 143.51 0)
@@
 	)
 	(symbol
-		(lib_name "Misc Keyboard Parts:SW_Kali_optional_reversable")
 		(lib_id "Misc Keyboard Parts:SW_Kali_optional_reversable")
 		(at 62.23 66.04 0)
@@
 	)
 	(symbol
-		(lib_name "Misc Keyboard Parts:SW_Kali_optional_reversable")
 		(lib_id "Misc Keyboard Parts:SW_Kali_optional_reversable")
 		(at 173.99 200.66 0)
@@
 	)
 	(symbol
-		(lib_name "Misc Keyboard Parts:SW_Kali_optional_reversable")
 		(lib_id "Misc Keyboard Parts:SW_Kali_optional_reversable")
 		(at 156.21 200.66 0)
@@
 	)
 	(symbol
-		(lib_name "Misc Keyboard Parts:SW_Kali_optional_reversable")
 		(lib_id "Misc Keyboard Parts:SW_Kali_optional_reversable")
 		(at 62.23 81.28 0)
@@
 	)
 	(symbol
-		(lib_name "Misc Keyboard Parts:SW_Kali_optional_reversable")
 		(lib_id "Misc Keyboard Parts:SW_Kali_optional_reversable")
 		(at 62.23 184.15 0)
@@
 	)
 	(symbol
-		(lib_name "Misc Keyboard Parts:SW_Kali_optional_reversable")
 		(lib_id "Misc Keyboard Parts:SW_Kali_optional_reversable")
 		(at 191.77 115.57 0)
@@
 	)
 	(symbol
-		(lib_name "Misc Keyboard Parts:SW_Kali_optional_reversable")
 		(lib_id "Misc Keyboard Parts:SW_Kali_optional_reversable")
 		(at 191.77 171.45 0)
@@
 	)
 	(symbol
-		(lib_name "Misc Keyboard Parts:SW_Kali_optional_reversable")
 		(lib_id "Misc Keyboard Parts:SW_Kali_optional_reversable")
 		(at 227.33 218.44 0)
@@
 	)
 	(symbol
-		(lib_name "Misc Keyboard Parts:SW_Kali_optional_reversable")
 		(lib_id "Misc Keyboard Parts:SW_Kali_optional_reversable")
 		(at 60.96 129.54 0)
@@
 	)
 	(symbol
-		(lib_name "Misc Keyboard Parts:SW_Kali_optional_reversable")
 		(lib_id "Misc Keyboard Parts:SW_Kali_optional_reversable")
 		(at 119.38 86.36 0)
@@
 	)
 	(symbol
-		(lib_name "Misc Keyboard Parts:SW_Kali_optional_reversable")
 		(lib_id "Misc Keyboard Parts:SW_Kali_optional_reversable")
 		(at 119.38 171.45 0)
@@
 	)
 	(symbol
-		(lib_name "Misc Keyboard Parts:SW_Kali_optional_reversable")
 		(lib_id "Misc Keyboard Parts:SW_Kali_optional_reversable")
 		(at 173.99 171.45 0)
@@
 	)
 	(symbol
-		(lib_name "Misc Keyboard Parts:SW_Kali_optional_reversable")
 		(lib_id "Misc Keyboard Parts:SW_Kali_optional_reversable")
 		(at 156.21 143.51 0)
@@
 	)
 	(symbol
-		(lib_name "Misc Keyboard Parts:SW_Kali_optional_reversable")
 		(lib_id "Misc Keyboard Parts:SW_Kali_optional_reversable")
 		(at 156.21 115.57 0)
@@
 	)
 	(symbol
-		(lib_name "Misc Keyboard Parts:SW_Kali_optional_reversable")
 		(lib_id "Misc Keyboard Parts:SW_Kali_optional_reversable")
 		(at 119.38 115.57 0)
@@
 	)
 	(symbol
-		(lib_name "Misc Keyboard Parts:SW_Kali_optional_reversable")
 		(lib_id "Misc Keyboard Parts:SW_Kali_optional_reversable")
 		(at 227.33 143.51 0)
@@
 	)
 	(symbol
-		(lib_name "Misc Keyboard Parts:SW_Kali_optional_reversable")
 		(lib_id "Misc Keyboard Parts:SW_Kali_optional_reversable")
 		(at 62.23 97.79 0)
@@
 	)
 	(symbol
-		(lib_name "Misc Keyboard Parts:SW_Kali_optional_reversable")
 		(lib_id "Misc Keyboard Parts:SW_Kali_optional_reversable")
 		(at 119.38 143.51 0)
@@
 	)
 	(symbol
-		(lib_name "Misc Keyboard Parts:SW_Kali_optional_reversable")
 		(lib_id "Misc Keyboard Parts:SW_Kali_optional_reversable")
 		(at 209.55 171.45 0)
@@
 	)
 	(symbol
-		(lib_name "Misc Keyboard Parts:SW_Kali_optional_reversable")
 		(lib_id "Misc Keyboard Parts:SW_Kali_optional_reversable")
 		(at 137.16 115.57 0)
@@
 	)
 	(symbol
-		(lib_name "Misc Keyboard Parts:SW_Kali_optional_reversable")
 		(lib_id "Misc Keyboard Parts:SW_Kali_optional_reversable")
 		(at 191.77 143.51 0)
@@
 	)
 	(symbol
-		(lib_name "Misc Keyboard Parts:SW_Kali_optional_reversable")
 		(lib_id "Misc Keyboard Parts:SW_Kali_optional_reversable")
 		(at 227.33 171.45 0)
@@
 	)
 	(symbol
-		(lib_name "Misc Keyboard Parts:SW_Kali_optional_reversable")
 		(lib_id "Misc Keyboard Parts:SW_Kali_optional_reversable")
 		(at 209.55 143.51 0)
@@
 	)
 	(symbol
-		(lib_name "Misc Keyboard Parts:SW_Kali_optional_reversable")
 		(lib_id "Misc Keyboard Parts:SW_Kali_optional_reversable")
 		(at 207.01 217.17 0)
@@
 	)
 	(symbol
-		(lib_name "Misc Keyboard Parts:SW_Kali_optional_reversable")
 		(lib_id "Misc Keyboard Parts:SW_Kali_optional_reversable")
 		(at 137.16 200.66 0)
@@
 	)
 	(symbol
-		(lib_name "Misc Keyboard Parts:SW_Kali_optional_reversable")
 		(lib_id "Misc Keyboard Parts:SW_Kali_optional_reversable")
 		(at 137.16 171.45 0)
@@
 	)
 	(symbol
-		(lib_name "Misc Keyboard Parts:SW_Kali_optional_reversable")
 		(lib_id "Misc Keyboard Parts:SW_Kali_optional_reversable")
 		(at 173.99 86.36 0)
@@
 	)
 	(symbol
-		(lib_name "Misc Keyboard Parts:SW_Kali_optional_reversable")
 		(lib_id "Misc Keyboard Parts:SW_Kali_optional_reversable")
 		(at 60.96 114.3 0)
@@
 	)
 	(symbol
-		(lib_name "Misc Keyboard Parts:SW_Kali_optional_reversable")
 		(lib_id "Misc Keyboard Parts:SW_Kali_optional_reversable")
 		(at 209.55 115.57 0)
@@
 	)
 	(symbol
-		(lib_name "Misc Keyboard Parts:SW_Kali_optional_reversable")
 		(lib_id "Misc Keyboard Parts:SW_Kali_optional_reversable")
 		(at 156.21 86.36 0)
@@
 	)
 	(symbol
-		(lib_name "Misc Keyboard Parts:SW_Kali_optional_reversable")
 		(lib_id "Misc Keyboard Parts:SW_Kali_optional_reversable")
 		(at 227.33 86.36 0)
@@
 	)
 	(symbol
-		(lib_name "Misc Keyboard Parts:SW_Kali_optional_reversable")
 		(lib_id "Misc Keyboard Parts:SW_Kali_optional_reversable")
 		(at 227.33 115.57 0)
@@
 	)
 	(symbol
-		(lib_name "Misc Keyboard Parts:SW_Kali_optional_reversable")
 		(lib_id "Misc Keyboard Parts:SW_Kali_optional_reversable")
 		(at 119.38 200.66 0)
@@
 	)
 	(symbol
-		(lib_name "Misc Keyboard Parts:SW_Kali_optional_reversable")
 		(lib_id "Misc Keyboard Parts:SW_Kali_optional_reversable")
 		(at 60.96 146.05 0)
@@
 	)
 	(symbol
-		(lib_name "Misc Keyboard Parts:SW_Kali_optional_reversable")
 		(lib_id "Misc Keyboard Parts:SW_Kali_optional_reversable")
 		(at 137.16 86.36 0)
@@
 	)
 	(symbol
-		(lib_name "Misc Keyboard Parts:SW_Kali_optional_reversable")
 		(lib_id "Misc Keyboard Parts:SW_Kali_optional_reversable")
 		(at 173.99 115.57 0)
@@
 	)
 	(symbol
-		(lib_name "Misc Keyboard Parts:SW_Kali_optional_reversable")
 		(lib_id "Misc Keyboard Parts:SW_Kali_optional_reversable")
 		(at 156.21 171.45 0)
